Commit message: first implementation of feetech servo hw interface

File: feetech_servo_bringup/urdf/feetech_servo.ros2_control.xacro (robot description, xacro)
@@ -13,25 +13,25 @@
                 >
         <ros2_control name="${name}" type="system">
-        <hardware>
-            <xacro:if value="${mock_hardware}">
-                <plugin>mock_components/GenericSystem</plugin>
-            </xacro:if>
-            <xacro:unless value="${mock_hardware}">
-                <plugin>feetech_servo_hardware_interface/FeetechServoHardwareInterface</plugin>
-                <param name="serial_port">${serial_port}</param>
-                <param name="baud_rate">${baud_rate}</param>
-                <param name="servo_id">${servo_id}</param>
-                <param name="servo_open_step">${servo_open_step}</param>
-                <param name="servo_closed_step">${servo_closed_step}</param>
-                <param name="gripper_open_pos">${gripper_open_pos}</param>
-                <param name="gripper_closed_pos">${gripper_closed_pos}</param>
-            </xacro:unless>
-        </hardware>
-        <gpio name="gripper">
-            <command_interface name="position"/>
-            <state_interface name="position"/>
-            <state_interface name="velocity"/>
-            <state_interface name="effort"/>
-        </gpio>
+            <hardware>
+                <xacro:if value="${mock_hardware}">
+                    <plugin>mock_components/GenericSystem</plugin>
+                </xacro:if>
+                <xacro:unless value="${mock_hardware}">
+                    <plugin>feetech_servo_hardware_interface/FeetechServoHardwareInterface</plugin>
+                    <param name="serial_port">${serial_port}</param>
+                    <param name="baud_rate">${baud_rate}</param>
+                    <param name="servo_id">${servo_id}</param>
+                    <param name="servo_open_step">${servo_open_step}</param>
+                    <param name="servo_closed_step">${servo_closed_step}</param>
+                    <param name="gripper_open_pos">${gripper_open_pos}</param>
+                    <param name="gripper_closed_pos">${gripper_closed_pos}</param>
+                </xacro:unless>
+            </hardware>
+            <joint name="gripper_joint">
+                <command_interface name="position"/>
+                <state_interface name="position"/>
+                <state_interface name="velocity"/>
+                <state_interface name="effort"/>
+            </joint>
         </ros2_control>
     </xacro:macro>

File: feetech_servo_bringup/urdf/feetech_test.urdf.xacro (robot description, xacro)
@@ -4,4 +4,17 @@
   <xacro:include filename="$(find feetech_servo_bringup)/urdf/feetech_servo.ros2_control.xacro"/>
   <link name="world"/>
+  <link name="link1"/>
+  <link name="link2"/>
+  <joint name="world-link1" type="fixed">
+    <parent link="world"/>
+    <child link="link1"/>
+    <limit effort="60" velocity="${radians(225)}" lower="${-2*pi}" upper="${2*pi}"/>
+  </joint>
+  <joint name="gripper_joint" type="revolute">
+    <parent link="link1"/>
+    <child link="link2"/>
+    <axis xyz="0 0 1"/>
+    <limit effort="60" velocity="${radians(225)}" lower="${-2*pi}" upper="${2*pi}"/>
+  </joint>
   <xacro:feetech_servo_ros2_control
     name="feetech_gripper"
