Commit message: make gripper_hand_joiint fixed - it is redundant w.r.t. Joint6

File: feetech_servo_bringup/urdf/feetech_gripper_macro.xacro (robot description, xacro)
@@ -36,5 +36,5 @@
     <joint
         name="GRIPPER_HAND_JOINT"
-        type="revolute">
+        type="fixed">
         <origin
         xyz="0 0.0 0"
@@ -44,11 +44,4 @@
         <child
         link="GRIPPER_HAND" />
-        <axis
-        xyz="0 0 1" />
-        <limit
-        lower="-6.28"
-        upper="6.28"
-        effort="0"
-        velocity="0.1" />
     </joint>
     <link
